File: pcb/mmwave/mmwave.kicad_sch (KiCad schematic)
At the start: 30 parts, among them J1 USB4105-GF-A, J2 PROG, J3 I2C, J4 MMW_SENSOR, J5 VIN, U1 AP7365-33ERG-13, U2 ESP32-C3-WROOM-02, U3 EKMB1305111K, U4 SHT4X, U5 N/A

Commit message: Updated BOM and schematic
Parts:
- U3: value EKMB1305111K -> EKMB1310111K
- U4: value SHT4X -> SHT45-AD1B-R2
Changed lines of the file:
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@@
   (title_block
     (title "Main board")
-    (date "2022-07-23")
-    (rev "A")
+    (date "2022-07-29")
+    (rev "B")
   )
   (junction (at 237.49 53.34) (diameter 0) (color 0 0 0 0)
@@
       (effects (font (size 1.524 1.524) bold) (justify left bottom))
     )
-    (property "Value" "EKMB1305111K" (id 1) (at 222.25 120.65 0)
+    (property "Value" "EKMB1310111K" (id 1) (at 222.25 120.65 0)
       (effects (font (size 1.016 1.016)) (justify left top))
     )
@@
       (effects (font (size 1.524 1.524) bold) (justify left bottom))
     )
-    (property "Value" "SHT4X" (id 1) (at 207.01 57.15 0)
+    (property "Value" "SHT45-AD1B-R2" (id 1) (at 207.01 57.15 0)
       (effects (font (size 1.016 1.016)) (justify left top))
     )
@@
     )
     (path "/2598b8aa-86d0-462c-8460-32c0cde63fbc"
-      (reference "U3") (unit 1) (value "EKMB1305111K") (footprint "misc:PIR-EKMB1310111K-EDGE")
+      (reference "U3") (unit 1) (value "EKMB1310111K") (footprint "misc:PIR-EKMB1310111K-EDGE")
     )
     (path "/a3348e31-db68-4af5-80ae-8b4b9734257d"
-      (reference "U4") (unit 1) (value "SHT4X") (footprint "smt-dfn:DFN4")
+      (reference "U4") (unit 1) (value "SHT45-AD1B-R2") (footprint "smt-dfn:DFN4")
     )
     (path "/ce420901-783b-4425-ad57-a5f8924f5a79"
